File: esp_testboard/HA_test.kicad_sch (KiCad schematic)
At the start: 105 parts, among them J1 ESP-01, J10 ESP-01, J11 SHT21, J12 SHT21, J13 SHT21, J14 SHT21, J15 SHT21, J16 PWR_IN, J17 629722000214, J18 UART, J2 ESP-01, J3 ESP-01, J4 ESP-01, J5 ESP-01, J6 ESP-01, J7 ESP-01, J8 ESP-01, J9 ESP-01, U1 AMS1117-3.3, U2 AMS1117-3.3

Commit message: finished test board for ESP
Parts:
- C1, C2, C3, C4: footprint Capacitor_SMD:C_1206_3216Metric -> Capacitor_SMD:C_0805_2012Metric
Other:
- note added: "USB-C"
Changed lines of the file:
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@@
   (title_block
     (title "ESP test board")
-    (date "2022-11-17")
+    (date "2022-11-27")
     (rev "1.0")
     (company "Paweł Jagowdzik")
-    (comment 1 "IN PROGRESS")
-    (comment 2 "IN PROGRESS")
-    (comment 3 "IN PROGRESS")
-    (comment 4 "IN PROGRESS")
+    (comment 2 "@pj_maker")
+    (comment 3 "github.com/Jadziu")
+    (comment 4 "paweljagowdzik@gmail.com")
   )
   (junction (at 87.63 39.37) (diameter 0) (color 0 0 0 0)
@@
     (stroke (width 0) (type default) (color 0 0 0 0))
   )
+  (polyline (pts (xy 215.9 90.17) (xy 279.4 90.17))
+    (stroke (width 0) (type default) (color 0 0 0 0))
+  )
   (wire (pts (xy 139.7 140.97) (xy 143.51 140.97))
     (stroke (width 0) (type default) (color 0 0 0 0))
@@
     (stroke (width 0) (type default) (color 0 0 0 0))
   )
+  (polyline (pts (xy 279.4 90.17) (xy 279.4 146.05))
+    (stroke (width 0) (type default) (color 0 0 0 0))
+  )
   (wire (pts (xy 190.5 133.35) (xy 193.04 133.35))
     (stroke (width 0) (type default) (color 0 0 0 0))
@@
     (stroke (width 0) (type default) (color 0 0 0 0))
   )
+  (polyline (pts (xy 279.4 146.05) (xy 215.9 146.05))
+    (stroke (width 0) (type default) (color 0 0 0 0))
+  )
   (wire (pts (xy 85.09 173.99) (xy 85.09 170.18))
     (stroke (width 0) (type default) (color 0 0 0 0))
@@
     (stroke (width 0) (type default) (color 0 0 0 0))
   )
+  (polyline (pts (xy 215.9 90.17) (xy 215.9 146.05))
+    (stroke (width 0) (type default) (color 0 0 0 0))
+  )
   (polyline (pts (xy 22.86 87.63) (xy 22.86 17.78))
     (stroke (width 0) (type default) (color 0 0 0 0))
@@
     (effects (font (size 2.54 2.54)) (justify left bottom))
   )
+  (text "USB-C" (at 218.44 143.51 0)
+    (effects (font (size 2.54 2.54)) (justify left bottom))
+  )
   (global_label "SCL3" (shape input) (at 107.95 167.64 0) (fields_autoplaced)
     (effects (font (size 1.27 1.27)) (justify left))
@@
       (effects (font (size 1.27 1.27)) (justify left))
     )
-    (property "Footprint" "Capacitor_SMD:C_1206_3216Metric" (id 2) (at 87.63 34.29 0)
+    (property "Footprint" "Capacitor_SMD:C_0805_2012Metric" (id 2) (at 87.63 34.29 0)
       (effects (font (size 1.27 1.27)) hide)
     )
@@
       (effects (font (size 1.27 1.27)) (justify left))
     )
-    (property "Footprint" "Capacitor_SMD:C_1206_3216Metric" (id 2) (at 87.63 60.96 0)
+    (property "Footprint" "Capacitor_SMD:C_0805_2012Metric" (id 2) (at 87.63 60.96 0)
       (effects (font (size 1.27 1.27)) hide)
     )
@@
       (effects (font (size 1.27 1.27)) (justify left))
     )
-    (property "Footprint" "Capacitor_SMD:C_1206_3216Metric" (id 2) (at 59.69 34.29 0)
+    (property "Footprint" "Capacitor_SMD:C_0805_2012Metric" (id 2) (at 59.69 34.29 0)
       (effects (font (size 1.27 1.27)) hide)
     )
@@
       (effects (font (size 1.27 1.27)) (justify left))
     )
-    (property "Footprint" "Capacitor_SMD:C_1206_3216Metric" (id 2) (at 59.69 60.96 0)
+    (property "Footprint" "Capacitor_SMD:C_0805_2012Metric" (id 2) (at 59.69 60.96 0)
       (effects (font (size 1.27 1.27)) hide)
     )
@@
     )
     (path "/9038cd39-bac3-469c-8317-1a22225eac73"
-      (reference "C1") (unit 1) (value "10uF") (footprint "Capacitor_SMD:C_1206_3216Metric")
+      (reference "C1") (unit 1) (value "10uF") (footprint "Capacitor_SMD:C_0805_2012Metric")
     )
     (path "/e7f8292e-7d23-42be-9e9c-f5760a3354a2"
-      (reference "C2") (unit 1) (value "10uF") (footprint "Capacitor_SMD:C_1206_3216Metric")
+      (reference "C2") (unit 1) (value "10uF") (footprint "Capacitor_SMD:C_0805_2012Metric")
     )
     (path "/678b99f9-ecce-4a59-b7d2-283f694bc917"
-      (reference "C3") (unit 1) (value "10uF") (footprint "Capacitor_SMD:C_1206_3216Metric")
+      (reference "C3") (unit 1) (value "10uF") (footprint "Capacitor_SMD:C_0805_2012Metric")
     )
     (path "/7758f5b4-73f0-4be6-91e8-94a3d930ea26"
-      (reference "C4") (unit 1) (value "10uF") (footprint "Capacitor_SMD:C_1206_3216Metric")
+      (reference "C4") (unit 1) (value "10uF") (footprint "Capacitor_SMD:C_0805_2012Metric")
     )
     (path "/ee970625-db62-415d-be10-35774b45d98e"
